File: blurf/main.sch (EAGLE design)
At the start: 5 parts

Commit message: antena added
Parts:
- added ANT1: JOHANSON868, mylib1:JOHANSON868
Changed lines of the file:
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@@
 <part name="PWR1" library="mylib1" deviceset="LT1767E-3.3" device=""/>
 <part name="CHGR1" library="mylib1" deviceset="MCP73837-FCI/UN" device=""/>
+<part name="ANT1" library="mylib1" deviceset="JOHANSON868" device=""/>
 </parts>
 <sheets>
@@
 <instance part="PWR1" gate="G$1" x="-139.7" y="-12.7"/>
 <instance part="CHGR1" gate="G$1" x="-127" y="50.8"/>
+<instance part="ANT1" gate="G$1" x="-139.7" y="114.3"/>
 </instances>
 <busses>
